File: radiohw/carrier/carrier.kicad_pcb (KiCad board)
At the start: 2 copper layers, 6 parts

Commit message: Unsaved changes.
Parts:
- added U3: ~, Package_DFN_QFN:QFN-40-1EP_5x5mm_P0.4mm_EP3.6x3.6mm_ThermalVias, F.Cu at (144.9, 99.8)
Connections:
- U1 pad 10: /ComExpressCarrier/GBE0_MDI1+ -> unconnected-(U1A-A10-Pad10)
- U1 pad 12: /ComExpressCarrier/GBE0_MDI0- -> unconnected-(U1A-A12-Pad12)
- U1 pad 13: /ComExpressCarrier/GBE0_MDI0+ -> unconnected-(U1A-A13-Pad13)
- U1 pad 2: /ComExpressCarrier/GBE0_MDI3- -> unconnected-(U1A-A2-Pad2)
- U1 pad 3: /ComExpressCarrier/GBE0_MDI3+ -> unconnected-(U1A-A3-Pad3)
- U1 pad 4: /ComExpressCarrier/GBE0_LNK100# -> unconnected-(U1A-A4-Pad4)
- U1 pad 5: /ComExpressCarrier/GBE0_LNK1000# -> unconnected-(U1A-A5-Pad5)
- U1 pad 6: /ComExpressCarrier/GBE0_MDI2- -> unconnected-(U1A-A6-Pad6)
- U1 pad 7: /ComExpressCarrier/GBE0_MDI2+ -> unconnected-(U1A-A7-Pad7)
- U1 pad 8: /ComExpressCarrier/GBE0_LINK# -> unconnected-(U1A-A8-Pad8)
- U1 pad 9: /ComExpressCarrier/GBE0_MDI1- -> unconnected-(U1A-A9-Pad9)
- U2 pad 125: unconnected-(U2B-B15-Pad125) -> Net-(J1-SCL)
- U2 pad 126: unconnected-(U2B-B16-Pad126) -> Net-(J1-SDA)
- U2 pad 136: unconnected-(U2B-B26-Pad136) -> Net-(J1-D2+)
- U2 pad 137: unconnected-(U2B-B27-Pad137) -> Net-(J1-D2-)
- U2 pad 139: unconnected-(U2B-B29-Pad139) -> Net-(J1-D1+)
- U2 pad 140: unconnected-(U2B-B30-Pad140) -> Net-(J1-D1-)
- U2 pad 142: unconnected-(U2B-B32-Pad142) -> Net-(J1-D0+)
- U2 pad 143: unconnected-(U2B-B33-Pad143) -> Net-(J1-D0-)
- U2 pad 146: unconnected-(U2B-B36-Pad146) -> Net-(J1-CK+)
- U2 pad 147: unconnected-(U2B-B37-Pad147) -> Net-(J1-CK-)
- U2 pad 24: unconnected-(U2A-A24-Pad24) -> Net-(J1-HPD)
