File: radiohw/carrier/untitled.kicad_sch (KiCad schematic)
At the start: 7 parts, among them J1 HDMI_A

Commit message: Update schematics.
Connections:
- net HDA_SYNC: now reaches U1.29 (A29)
- net HDA_RST#: now reaches U1.30 (A30)
- net HDA_BITCLK: now reaches U1.32 (A32)
- net HDA_SDOUT: now reaches U1.33 (A33)
- net HDA_SDIN0: now reaches U1.140 (B30)
Changed lines of the file:
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@@
+    (stroke (width 0) (type default))
+  )
+  (wire (pts (xy 102.87 26.67) (xy 102.87 31.75))
     (stroke (width 0) (type default))
   )
@@
     (stroke (width 0) (type default))
   )
+  (wire (pts (xy 97.79 71.12) (xy 97.79 76.2))
+    (stroke (width 0) (type default))
+  )
   (wire (pts (xy 85.09 49.53) (xy 85.09 53.34))
     (stroke (width 0) (type default))
@@
     (stroke (width 0) (type default))
   )
+  (wire (pts (xy 95.25 26.67) (xy 95.25 31.75))
+    (stroke (width 0) (type default))
+  )
   (wire (pts (xy 194.31 125.73) (xy 198.12 125.73))
     (stroke (width 0) (type default))
@@
     (stroke (width 0) (type default))
   )
+  (wire (pts (xy 97.79 26.67) (xy 97.79 31.75))
+    (stroke (width 0) (type default))
+  )
   (wire (pts (xy 86.36 143.51) (xy 182.88 143.51))
     (stroke (width 0) (type default))
@@
     (stroke (width 0) (type default))
   )
+  (wire (pts (xy 105.41 26.67) (xy 105.41 31.75))
+    (stroke (width 0) (type default))
+  )
   (wire (pts (xy 114.3 152.4) (xy 194.31 152.4))
     (stroke (width 0) (type default))
@@
     (stroke (width 0) (type default))
   )
+  (global_label "HDA_RST#" (shape input) (at 97.79 26.67 90) (fields_autoplaced)
+    (effects (font (size 1.27 1.27)) (justify left))
+    (property "Intersheetrefs" "${INTERSHEET_REFS}" (at 97.79 14.311 90)
+      (effects (font (size 1.27 1.27)) (justify left) hide)
+    )
+  )
+  (global_label "HDA_SDIN0" (shape input) (at 97.79 71.12 90) (fields_autoplaced)
+    (effects (font (size 1.27 1.27)) (justify left))
+    (property "Intersheetrefs" "${INTERSHEET_REFS}" (at 97.79 57.8538 90)
+      (effects (font (size 1.27 1.27)) (justify left) hide)
+    )
+  )
+  (global_label "HDA_SDOUT" (shape input) (at 105.41 26.67 90) (fields_autoplaced)
+    (effects (font (size 1.27 1.27)) (justify left))
+    (property "Intersheetrefs" "${INTERSHEET_REFS}" (at 105.41 12.92 90)
+      (effects (font (size 1.27 1.27)) (justify left) hide)
+    )
+  )
+  (global_label "PCBEEP" (shape input) (at 198.12 54.61 180) (fields_autoplaced)
+    (effects (font (size 1.27 1.27)) (justify right))
+    (property "Intersheetrefs" "${INTERSHEET_REFS}" (at 187.7568 54.61 0)
+      (effects (font (size 1.27 1.27)) (justify right) hide)
+    )
+  )
+  (global_label "HDA_BITCLK" (shape input) (at 102.87 26.67 90) (fields_autoplaced)
+    (effects (font (size 1.27 1.27)) (justify left))
+    (property "Intersheetrefs" "${INTERSHEET_REFS}" (at 102.87 12.6176 90)
+      (effects (font (size 1.27 1.27)) (justify left) hide)
+    )
+  )
+  (global_label "HDA_SYNC" (shape input) (at 95.25 26.67 90) (fields_autoplaced)
+    (effects (font (size 1.27 1.27)) (justify left))
+    (property "Intersheetrefs" "${INTERSHEET_REFS}" (at 95.25 14.1295 90)
+      (effects (font (size 1.27 1.27)) (justify left) hide)
+    )
+  )
   (symbol (lib_id "Mechanical:MountingHole_Pad") (at 264.16 20.32 0) (unit 1)

Commit message: Schematic development.
Connections:
- net GND: now also U1.111 (B1), U1.121 (B11), U1.131 (B21), U1.141 (B31), U1.151 (B41), U1.161 (B51), U1.170 (B60), U1.180 (B70), U1.190 (B80), U1.200 (B90), U1.210 (B100), U1.220 (B110), U1.57 (A57), U2.1 (A1), U2.100 (A100), U2.11 (A11), U2.110 (A110), U2.111 (B1), U2.121 (B11), U2.131 (B21), U2.141 (B31), U2.151 (B41), U2.161 (B51), U2.170 (B60), U2.180 (B70), U2.190 (B80), U2.200 (B90), U2.21 (A21), U2.210 (B100), U2.220 (B110), U2.31 (A31), U2.41 (A41), U2.51 (A51), U2.60 (A60), U2.70 (A70), U2.80 (A80), U2.90 (A90)
- net WIRELESS_PCIE_TX0+: now reaches U1.55 (A55)
- net WIRELESS_PCIE_TX0-: now reaches U1.56 (A56)
- net STORAGE_PCIE_TX3+: now reaches U1.58 (A58)
- net STORAGE_PCIE_TX3-: now reaches U1.59 (A59)
- net STORAGE_PCIE_TX2+: now reaches U1.61 (A61)
- net STORAGE_PCIE_TX2-: now reaches U1.62 (A62)
- net STORAGE_PCIE_TX1+: now reaches U1.64 (A64)
- net STORAGE_PCIE_TX1-: now reaches U1.65 (A65)
- net STORAGE_PCIE_TX0+: now reaches U1.68 (A68)
- net STORAGE_PCIE_TX0-: now reaches U1.69 (A69)
- net SCL: now reaches U1.143 (B33)
- net SDA: now reaches U1.144 (B34)
- net WIRELESS_PCIE_RX0+: now reaches U1.165 (B55)
- net WIRELESS_PCIE_RX0-: now reaches U1.166 (B56)
- net STORAGE_PCIE_RX3+: now reaches U1.168 (B58)
- net STORAGE_PCIE_RX3-: now reaches U1.169 (B59)
- net STORAGE_PCIE_RX2+: now reaches U1.171 (B61)
- net STORAGE_PCIE_RX2-: now reaches U1.172 (B62)
- net STORAGE_PCIE_RX1-: now reaches U1.174 (B64)
- net STORAGE_PCIE_RX1+: now reaches U1.175 (B65)
- net STORAGE_PCIE_RX0+: now reaches U1.178 (B68)
- net STORAGE_PCIE_RX0-: now reaches U1.179 (B69)
