File: radiohw/carrier/dual_speaker.kicad_sch (KiCad schematic)
At the start: 10 parts, among them U12 E-TDA7560

Commit message: Audio schematic development.
Changed lines of the file:
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@@
   )
   (symbol (lib_id "Device:C") (at 110.49 100.33 90) (unit 1)
-    (in_bom yes) (on_board yes) (dnp no) (fields_autoplaced)
-    (property "Reference" "C10" (at 110.49 92.71 90)
-      (effects (font (size 1.27 1.27)))
-    )
-    (property "Value" "100nF" (at 110.49 95.25 90)
+    (in_bom yes) (on_board yes) (dnp no)
+    (property "Reference" "C10" (at 106.68 99.06 90)
+      (effects (font (size 1.27 1.27)))
+    )
+    (property "Value" "100nF" (at 114.3 99.06 90)
       (effects (font (size 1.27 1.27)))
     )
@@
   (symbol (lib_id "Device:C") (at 134.62 123.19 0) (unit 1)
     (in_bom yes) (on_board yes) (dnp no)
-    (property "Reference" "C12" (at 138.43 127 0)
-      (effects (font (size 1.27 1.27)) (justify left))
-    )
-    (property "Value" "47uF" (at 138.43 129.54 0)
+    (property "Reference" "C12" (at 129.54 120.65 0)
+      (effects (font (size 1.27 1.27)) (justify left))
+    )
+    (property "Value" "47uF" (at 129.54 125.73 0)
       (effects (font (size 1.27 1.27)) (justify left))
     )
@@
   )
   (symbol (lib_id "Device:C") (at 124.46 123.19 0) (unit 1)
-    (in_bom yes) (on_board yes) (dnp no) (fields_autoplaced)
-    (property "Reference" "C19" (at 128.27 121.92 0)
-      (effects (font (size 1.27 1.27)) (justify left))
-    )
-    (property "Value" "470nF" (at 128.27 124.46 0)
+    (in_bom yes) (on_board yes) (dnp no)
+    (property "Reference" "C19" (at 119.38 120.65 0)
+      (effects (font (size 1.27 1.27)) (justify left))
+    )
+    (property "Value" "470nF" (at 118.11 125.73 0)
       (effects (font (size 1.27 1.27)) (justify left))
     )
@@
   )
   (symbol (lib_id "Device:C") (at 110.49 88.9 90) (unit 1)
-    (in_bom yes) (on_board yes) (dnp no) (fields_autoplaced)
-    (property "Reference" "C15" (at 110.49 81.28 90)
-      (effects (font (size 1.27 1.27)))
-    )
-    (property "Value" "100nF" (at 110.49 83.82 90)
+    (in_bom yes) (on_board yes) (dnp no)
+    (property "Reference" "C15" (at 106.68 87.63 90)
+      (effects (font (size 1.27 1.27)))
+    )
+    (property "Value" "100nF" (at 114.3 87.63 90)
       (effects (font (size 1.27 1.27)))
     )
@@
   )
   (symbol (lib_id "Device:R_US") (at 172.72 71.12 90) (unit 1)
-    (in_bom yes) (on_board yes) (dnp no) (fields_autoplaced)
-    (property "Reference" "R18" (at 172.72 64.77 90)
-      (effects (font (size 1.27 1.27)))
-    )
-    (property "Value" "10k" (at 172.72 67.31 90)
+    (in_bom yes) (on_board yes) (dnp no)
+    (property "Reference" "R18" (at 172.72 66.04 90)
+      (effects (font (size 1.27 1.27)))
+    )
+    (property "Value" "10k" (at 172.72 68.58 90)
       (effects (font (size 1.27 1.27)))
     )
@@
   )
   (symbol (lib_id "Device:C") (at 110.49 96.52 90) (unit 1)
-    (in_bom yes) (on_board yes) (dnp no) (fields_autoplaced)
-    (property "Reference" "C9" (at 110.49 88.9 90)
-      (effects (font (size 1.27 1.27)))
-    )
-    (property "Value" "100nF" (at 110.49 91.44 90)
+    (in_bom yes) (on_board yes) (dnp no)
+    (property "Reference" "C9" (at 106.68 95.25 90)
+      (effects (font (size 1.27 1.27)))
+    )
+    (property "Value" "100nF" (at 114.3 95.25 90)
       (effects (font (size 1.27 1.27)))
     )
@@
   )
   (symbol (lib_id "Device:C") (at 110.49 92.71 90) (unit 1)
-    (in_bom yes) (on_board yes) (dnp no) (fields_autoplaced)
-    (property "Reference" "C8" (at 110.49 85.09 90)
-      (effects (font (size 1.27 1.27)))
-    )
-    (property "Value" "100nF" (at 110.49 87.63 90)
-      (effects (font (size 1.27 1.27)))
-    )
+    (in_bom yes) (on_board yes) (dnp no)
+    (property "Reference" "C8" (at 106.68 91.44 90)
+      (effects (font (size 1.27 1.27)))
+    )
+    (property "Value" "100nF" (at 114.3 91.44 90)
+      (effects (font (size 1.27 1.27)))
+    )
